File: hardware/kicad/esp32-tallighty.kicad_pcb (KiCad board)
At the start: 2 copper layers, 65 x 35 mm, 10 parts, among them SW1 SW_Push, SW2 SW_Push, SW3 SW_Push, U1 ESP32-C3_SUPERMINI_TH

Commit message: update kicad project
Parts:
- added C1: 100n, Capacitor_SMD:C_1206_3216Metric, B.Cu at (150.5, 129.0)
- added C2: 100n, Capacitor_SMD:C_1206_3216Metric, B.Cu at (133.2, 129.0)
- added R1: 100, Resistor_SMD:R_1206_3216Metric, B.Cu at (137.0, 126.5)
- added R2: 100, Resistor_SMD:R_1206_3216Metric, B.Cu at (142.0, 126.5)
- added R3: 100, Resistor_SMD:R_1206_3216Metric, B.Cu at (147.0, 126.5)
- added R4: 100, Resistor_SMD:R_1206_3216Metric, B.Cu at (137.0, 130.0)
- added R5: 100, Resistor_SMD:R_1206_3216Metric, B.Cu at (142.0, 130.0)
- added R6: 100, Resistor_SMD:R_1206_3216Metric, B.Cu at (147.0, 130.0)
- moved U1 0.50 mm to (123.0, 117.0)
Connections:
- U1 pad 20: Net-(D1-DIN) -> Net-(U1-GPIO20)
- U1 pad 21: Net-(D2-DIN) -> Net-(U1-GPIO21)
Routing:
- net Net-(U1-GPIO3): track 0.00 -> 55.3 mm
- net Net-(U1-GPIO1): track 0.00 -> 45.5 mm
- net Net-(U1-GPIO0): track 0.00 -> 40.2 mm
- net Net-(D2-DIN): track 0.00 -> 27.9 mm
- net Net-(D1-DIN): track 0.00 -> 12.1 mm
- net Net-(U1-GPIO20): track 0.00 -> 9.11 mm
- net Net-(U1-GPIO21): track 0.00 -> 8.56 mm
- net Net-(R5-Pad1): track 0.00 -> 2.07 mm
- net Net-(R4-Pad1): track 0.00 -> 2.07 mm
- net Net-(R2-Pad1): track 0.00 -> 2.07 mm
- net Net-(R1-Pad1): track 0.00 -> 2.07 mm
- net VBUS: vias 0 -> 2
Other:
- board text added: "Design By RioLi"
- board text added: "ESP32-Tallighty"
- board text added: "Hold [SET] 1s to open Menu. Click [SET] to Edit/Save values. * Auto-exits menu after 5s idle. * Hotspot: Tallighty-Setup * Password: 13051368"
