File: hardware/kicad/esp32-tallighty.kicad_sch (KiCad schematic)
At the start: 10 parts, among them SW1 SW_Push, SW2 SW_Push, SW3 SW_Push, U1 ESP32-C3_SUPERMINI_TH

Commit message: update kicad project
Parts:
- added C1, C2: 100n, Capacitor_SMD:C_1206_3216Metric, symbol Device:C
- added R1, R2, R3, R4, R5, R6: 100, Resistor_SMD:R_1206_3216Metric, symbol Device:R
Connections:
- net GND: now also C1.2, C2.2
- net VBUS: now also C1.1, C2.1
- net at U1.20 (GPIO20): now also R1.2; no longer D1.4 (DIN)
- net at D2.4 (DIN): now also R6.1; no longer U1.21 (GPIO21)
- new net: R5.1, R6.2
- new net: R2.1, R3.2
- new net: R1.1, R2.2
- new net: R4.1, R5.2
- new net: R4.2, U1.21 (GPIO21)
- new net: D1.4 (DIN), R3.1
